Commit message: 仿真联调：修复 Gazebo 闪退/控制器加载/机械臂抬升，忽略构建产物
- 修复 Gazebo GUI 闪退：清理 snap 环境变量（GTK_PATH 等），移除软件渲染
- 修复 arm_group_controller spawner 锁竞争：合并为单 spawner
- ros2_control 标签提升为 URDF 顶层，controller_manager 由 Gazebo 插件拉起
- 机械臂抬升：位置接口比例增益默认 0.1 太弱，增至 0.5
- URDF 关节 limit effort/velocity 由 0 改为有效值
- move_group 显式 use_sim_time，rviz 直传 robot_description_semantic
- ompl_planning.yaml 适配 MoveIt2 新格式
- 重写 README_SIM.md，更新项目介绍.md，新增项目修改记录.md
- 新增 .gitignore，将 build/install/log 构建产物移出版本控制

File: src/episode1_moveit_config/config/episode1_urdf_1113.ros2_control.xacro (robot description, xacro)
@@ -3,14 +3,18 @@
     <xacro:macro name="episode1_urdf_1113_ros2_control" params="name initial_positions_file">
         <xacro:property name="initial_positions" value="${xacro.load_yaml(initial_positions_file)['initial_positions']}"/>
-        <gazebo>
-            <plugin filename="gz_ros2_control-system" name="gz_ros2_control::GazeboSimROS2ControlPlugin">
-                <ros2_control name="${name}" type="system">
-                    <hardware>
-                        <plugin>gz_ros2_control/GazeboSimSystem</plugin>
-                    </hardware>
+        <!-- ros2_control 硬件接口定义：必须是 <robot> 的直接子元素（顶层）。
+             Gazebo 进程内的 controller_manager 通过 /robot_description 话题
+             收到 URDF 后，用 parse_urdf 读取顶层的 <ros2_control> 标签来初始化
+             GazeboSimSystem 硬件接口。若把它嵌套在 <gazebo><plugin> 里，会被
+             URDF 解析器当成 gazebo 扩展而忽略，从而报
+             "no 'ros2_control' tag found in the URDF"。 -->
+        <ros2_control name="${name}" type="system">
+            <hardware>
+                <plugin>gz_ros2_control/GazeboSimSystem</plugin>
+            </hardware>
             <joint name="joint1">
                 <command_interface name="position"/>
                 <state_interface name="position">
-                  <param name="initial_value">${initial_positions['joint1']}</param>
+                    <param name="initial_value">${initial_positions['joint1']}</param>
                 </state_interface>
                 <state_interface name="velocity"/>
@@ -19,5 +23,5 @@
                 <command_interface name="position"/>
                 <state_interface name="position">
-                  <param name="initial_value">${initial_positions['joint2']}</param>
+                    <param name="initial_value">${initial_positions['joint2']}</param>
                 </state_interface>
                 <state_interface name="velocity"/>
@@ -26,5 +30,5 @@
                 <command_interface name="position"/>
                 <state_interface name="position">
-                  <param name="initial_value">${initial_positions['joint3']}</param>
+                    <param name="initial_value">${initial_positions['joint3']}</param>
                 </state_interface>
                 <state_interface name="velocity"/>
@@ -33,5 +37,5 @@
                 <command_interface name="position"/>
                 <state_interface name="position">
-                  <param name="initial_value">${initial_positions['joint4']}</param>
+                    <param name="initial_value">${initial_positions['joint4']}</param>
                 </state_interface>
                 <state_interface name="velocity"/>
@@ -40,5 +44,5 @@
                 <command_interface name="position"/>
                 <state_interface name="position">
-                  <param name="initial_value">${initial_positions['joint5']}</param>
+                    <param name="initial_value">${initial_positions['joint5']}</param>
                 </state_interface>
                 <state_interface name="velocity"/>
@@ -47,9 +51,20 @@
                 <command_interface name="position"/>
                 <state_interface name="position">
-                  <param name="initial_value">${initial_positions['joint6']}</param>
+                    <param name="initial_value">${initial_positions['joint6']}</param>
                 </state_interface>
                 <state_interface name="velocity"/>
             </joint>
-                </ros2_control>
+        </ros2_control>
+        <!-- Gazebo 插件：负责 (1) 在 Gazebo 进程内实例化 controller_manager、
+             (2) 从 <parameters> 加载控制器配置（update_rate + 控制器定义）。
+             硬件接口定义在上面的顶层 <ros2_control> 里，经 /robot_description
+             话题送达 Gazebo 内的 controller_manager，二者相互独立。 -->
+        <gazebo>
+            <plugin filename="gz_ros2_control-system" name="gz_ros2_control::GazeboSimROS2ControlPlugin">
+                <parameters>$(find episode1_moveit_config)/config/ros2_controllers.yaml</parameters>
+                <!-- 位置指令接口的比例增益（默认 0.1 太弱，扛不住重力，机械臂抬不起来）。
+                     增益越大跟踪越快，但 <=1 才不振荡、<=2 才稳定。
+                     joint_velocity = gain * position_error * update_rate（update_rate=100）。 -->
+                <position_proportional_gain>0.5</position_proportional_gain>
             </plugin>
         </gazebo>

File: src/episode1_urdf_1113/urdf/episode1_urdf_1113.urdf (robot description, URDF)
Before this commit: robot episode1_urdf_1113, 7 links, 6 joints
Joints:
- joint joint1: limit lower=-3.141592654 upper=2.792526803 effort=0 velocity=0 -> lower=-3.141592654 upper=2.792526803 effort=100 velocity=6.28
- joint joint2: limit lower=-1.570796327 upper=1.570796327 effort=0 velocity=0 -> lower=-1.570796327 upper=1.570796327 effort=100 velocity=6.28
- joint joint3: limit lower=-1.448623279 upper=1.396263402 effort=0 velocity=0 -> lower=-1.448623279 upper=1.396263402 effort=100 velocity=6.28
- joint joint4: limit lower=-0.523598776 upper=5.323254219 effort=0 velocity=0 -> lower=-0.523598776 upper=5.323254219 effort=100 velocity=6.28
- joint joint5: limit lower=-1.919862177 upper=1.919862177 effort=0 velocity=0 -> lower=-1.919862177 upper=1.919862177 effort=100 velocity=6.28
- joint joint6: limit lower=-0.523598776 upper=5.323254219 effort=0 velocity=0 -> lower=-0.523598776 upper=5.323254219 effort=100 velocity=6.28
